Commit message: fdfb

File: staubli_tx2_90_description/urdf/staubli_tx2_90_support.urdf.xacro (robot description, xacro)
@@ -13,14 +13,14 @@
       <origin rpy="0 0 0" xyz="0 0 0"/>
       <geometry>
-        <mesh filename="package://staubli_tx2_90_support/meshes/tx2_90/visual/base_link.stl"/>
-      </geometry>
-      <material name="">
-        <color rgba="1.0 0.6078431372549019 0.0 1.0"/>
-      </material>
-    </visual>
-    <collision>
-      <origin rpy="0 0 0" xyz="0 0 0"/>
-      <geometry>
-        <mesh filename="package://staubli_tx2_90_support/meshes/tx2_90/collision/base_link.stl"/>
+        <mesh filename="package://staubli_tx2_90_description/meshes/tx2_90/visual/base_link.stl"/>
+      </geometry>
+      <material name="">
+        <color rgba="1.0 0.6078431372549019 0.0 1.0"/>
+      </material>
+    </visual>
+    <collision>
+      <origin rpy="0 0 0" xyz="0 0 0"/>
+      <geometry>
+        <mesh filename="package://staubli_tx2_90_description/meshes/tx2_90/collision/base_link.stl"/>
       </geometry>
     </collision>
@@ -30,14 +30,14 @@
       <origin rpy="0 0 0" xyz="0 0 0"/>
       <geometry>
-        <mesh filename="package://staubli_tx2_90_support/meshes/tx2_90/visual/link_1.stl"/>
-      </geometry>
-      <material name="">
-        <color rgba="1.0 0.6078431372549019 0.0 1.0"/>
-      </material>
-    </visual>
-    <collision>
-      <origin rpy="0 0 0" xyz="0 0 0"/>
-      <geometry>
-        <mesh filename="package://staubli_tx2_90_support/meshes/tx2_90/collision/link_1.stl"/>
+        <mesh filename="package://staubli_tx2_90_description/meshes/tx2_90/visual/link_1.stl"/>
+      </geometry>
+      <material name="">
+        <color rgba="1.0 0.6078431372549019 0.0 1.0"/>
+      </material>
+    </visual>
+    <collision>
+      <origin rpy="0 0 0" xyz="0 0 0"/>
+      <geometry>
+        <mesh filename="package://staubli_tx2_90_description/meshes/tx2_90/collision/link_1.stl"/>
       </geometry>
     </collision>
@@ -47,14 +47,14 @@
       <origin rpy="0 0 0" xyz="0 0 0"/>
       <geometry>
-        <mesh filename="package://staubli_tx2_90_support/meshes/tx2_90/visual/link_2.stl"/>
-      </geometry>
-      <material name="">
-        <color rgba="1.0 0.6078431372549019 0.0 1.0"/>
-      </material>
-    </visual>
-    <collision>
-      <origin rpy="0 0 0" xyz="0 0 0"/>
-      <geometry>
-        <mesh filename="package://staubli_tx2_90_support/meshes/tx2_90/collision/link_2.stl"/>
+        <mesh filename="package://staubli_tx2_90_description/meshes/tx2_90/visual/link_2.stl"/>
+      </geometry>
+      <material name="">
+        <color rgba="1.0 0.6078431372549019 0.0 1.0"/>
+      </material>
+    </visual>
+    <collision>
+      <origin rpy="0 0 0" xyz="0 0 0"/>
+      <geometry>
+        <mesh filename="package://staubli_tx2_90_description/meshes/tx2_90/collision/link_2.stl"/>
       </geometry>
     </collision>
@@ -64,14 +64,14 @@
       <origin rpy="0 0 0" xyz="0 0 0"/>
       <geometry>
-        <mesh filename="package://staubli_tx2_90_support/meshes/tx2_90/visual/link_3.stl"/>
-      </geometry>
-      <material name="">
-        <color rgba="1.0 0.6078431372549019 0.0 1.0"/>
-      </material>
-    </visual>
-    <collision>
-      <origin rpy="0 0 0" xyz="0 0 0"/>
-      <geometry>
-        <mesh filename="package://staubli_tx2_90_support/meshes/tx2_90/collision/link_3.stl"/>
+        <mesh filename="package://staubli_tx2_90_description/meshes/tx2_90/visual/link_3.stl"/>
+      </geometry>
+      <material name="">
+        <color rgba="1.0 0.6078431372549019 0.0 1.0"/>
+      </material>
+    </visual>
+    <collision>
+      <origin rpy="0 0 0" xyz="0 0 0"/>
+      <geometry>
+        <mesh filename="package://staubli_tx2_90_description/meshes/tx2_90/collision/link_3.stl"/>
       </geometry>
     </collision>
@@ -81,14 +81,14 @@
       <origin rpy="0 0 0" xyz="0 0 0"/>
       <geometry>
-        <mesh filename="package://staubli_tx2_90_support/meshes/tx2_90/visual/link_4.stl"/>
-      </geometry>
-      <material name="">
-        <color rgba="1.0 0.6078431372549019 0.0 1.0"/>
-      </material>
-    </visual>
-    <collision>
-      <origin rpy="0 0 0" xyz="0 0 0"/>
-      <geometry>
-        <mesh filename="package://staubli_tx2_90_support/meshes/tx2_90/collision/link_4.stl"/>
+        <mesh filename="package://staubli_tx2_90_description/meshes/tx2_90/visual/link_4.stl"/>
+      </geometry>
+      <material name="">
+        <color rgba="1.0 0.6078431372549019 0.0 1.0"/>
+      </material>
+    </visual>
+    <collision>
+      <origin rpy="0 0 0" xyz="0 0 0"/>
+      <geometry>
+        <mesh filename="package://staubli_tx2_90_description/meshes/tx2_90/collision/link_4.stl"/>
       </geometry>
     </collision>
@@ -98,5 +98,5 @@
       <origin rpy="0 0 0" xyz="0 0 0"/>
       <geometry>
-        <mesh filename="package://staubli_tx2_90_support/meshes/tx2_90/visual/link_5.stl"/>
+        <mesh filename="package://staubli_tx2_90_description/meshes/tx2_90/visual/link_5.stl"/>
       </geometry>
       <material name="">
@@ -107,5 +107,5 @@
       <origin rpy="0 0 0" xyz="0 0 0"/>
       <geometry>
-        <mesh filename="package://staubli_tx2_90_support/meshes/tx2_90/collision/link_5.stl"/>
+        <mesh filename="package://staubli_tx2_90_description/meshes/tx2_90/collision/link_5.stl"/>
       </geometry>
     </collision>
@@ -115,5 +115,5 @@
       <origin rpy="0 0 0" xyz="0 0 0"/>
       <geometry>
-        <mesh filename="package://staubli_tx2_90_support/meshes/tx2_90/visual/link_6.stl"/>
+        <mesh filename="package://staubli_tx2_90_description/meshes/tx2_90/visual/link_6.stl"/>
       </geometry>
       <material name="">
@@ -124,5 +124,5 @@
       <origin rpy="0 0 0" xyz="0 0 0"/>
       <geometry>
-        <mesh filename="package://staubli_tx2_90_support/meshes/tx2_90/collision/link_6.stl"/>
+        <mesh filename="package://staubli_tx2_90_description/meshes/tx2_90/collision/link_6.stl"/>
       </geometry>
     </collision>

File: staubli_tx2_90_description/urdf/tx2_90l.urdf (robot description, URDF)
Before this commit: robot staubli_tx2_90l, 10 links, 9 joints
Links:
- link base_link: geometry collision mesh filename=package://staubli_tx2_90_description/meshes/tx2_90/collisio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; visual mesh filename=package://staubli_tx2_90_description/meshes/tx2_90/visual/b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
- link link_1: geometry collision mesh filename=package://staubli_tx2_90_description/meshes/tx2_90/collisio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; visual mesh filename=package://staubli_tx2_90_description/meshes/tx2_90/visual/l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
- link link_2: geometry collision mesh filename=package://staubli_tx2_90_description/meshes/tx2_90l/collisi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; visual mesh filename=package://staubli_tx2_90_description/meshes/tx2_90l/visual/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
- link link_3: geometry collision mesh filename=package://staubli_tx2_90_description/meshes/tx2_90/collisio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; visual mesh filename=package://staubli_tx2_90_description/meshes/tx2_90/visual/l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
- link link_4: geometry collision mesh filename=package://staubli_tx2_90_description/meshes/tx2_90l/collisi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; visual mesh filename=package://staubli_tx2_90_description/meshes/tx2_90l/visual/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
- link link_5: geometry collision mesh filename=package://staubli_tx2_90_description/meshes/tx2_90/collisio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; visual mesh filename=package://staubli_tx2_90_description/meshes/tx2_90/visual/l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
- link link_6: geometry collision mesh filename=package://staubli_tx2_90_description/meshes/tx2_90/collisio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; visual mesh filename=package://staubli_tx2_90_description/meshes/tx2_90/visual/l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

File: staubli_tx2_90_description/urdf/tx2_90xl.urdf (robot description, URDF)
Before this commit: robot staubli_tx2_90xl, 10 links, 9 joints
Links:
- link base_link: geometry collision mesh filename=package://staubli_tx2_90_description/meshes/tx2_90/collisio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; visual mesh filename=package://staubli_tx2_90_description/meshes/tx2_90/visual/b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
- link link_1: geometry collision mesh filename=package://staubli_tx2_90_description/meshes/tx2_90/collisio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; visual mesh filename=package://staubli_tx2_90_description/meshes/tx2_90/visual/l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
- link link_2: geometry collision mesh filename=package://staubli_tx2_90_description/meshes/tx2_90xl/collis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; visual mesh filename=package://staubli_tx2_90_description/meshes/tx2_90xl/visual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
- link link_3: geometry collision mesh filename=package://staubli_tx2_90_description/meshes/tx2_90/collisio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; visual mesh filename=package://staubli_tx2_90_description/meshes/tx2_90/visual/l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
- link link_4: geometry collision mesh filename=package://staubli_tx2_90_description/meshes/tx2_90xl/collis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; visual mesh filename=package://staubli_tx2_90_description/meshes/tx2_90xl/visual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
- link link_5: geometry collision mesh filename=package://staubli_tx2_90_description/meshes/tx2_90/collisio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; visual mesh filename=package://staubli_tx2_90_description/meshes/tx2_90/visual/l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
- link link_6: geometry collision mesh filename=package://staubli_tx2_90_description/meshes/tx2_90/collisio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; visual mesh filename=package://staubli_tx2_90_description/meshes/tx2_90/visual/l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
